Commit message: update to v2 compatible

File: urdfs/mc_one.urdf (robot description, URDF)
Before this commit: robot mc_one, 55 links, 57 joints
Links:
- removed link base
- removed link chest_camera
- added link base_link; visual mesh filename=package://mc_robot_description/meshes/mc_one/base.stl
- added link chest_camera_link; visual mesh filename=package://mc_robot_description/meshes/mc_one/camera.stl
Joints:
- joint _wheel_middle: parent base -> base_link
- joint camera_sensor_joint: parent chest_camera -> chest_camera_link
- joint chest_camera: child chest_camera -> chest_camera_link
- joint knees: parent base -> base_link

Commit message: update urdf,change base_link

File: urdfs/mc_one.urdf (robot description, URDF)
Before this commit: robot mc_one, 55 links, 57 joints
Links:
- removed link wheel_middle
Joints:
- removed joint _wheel_middle
- joint chest_camera: origin xyz=0.048749 0 0.3 rpy=0 0 0 -> xyz=0.048749 0 0.336 rpy=0 0 0
- joint hips: limit lower=0.3665 upper=-1.5708 effort=0 velocity=0 -> lower=-0.3665 upper=1.5708 effort=0 velocity=0; mimic (none) -> joint=knees multiplier=-1 offset=0
- joint knees: origin xyz=-0.0275 0 0.302 rpy=0 0 0 -> xyz=-0.0275 0 0.226 rpy=0 0 0
- joint left_wheel: parent wheel_middle -> base_link
- joint right_wheel: parent wheel_middle -> base_link

Commit message: fixed right hand, add laser

File: urdfs/mc_one.urdf (robot description, URDF)
Before this commit: robot mc_one, 54 links, 56 joints
Links:
- added link laser
Joints:
- added joint laser_mount: type fixed, parent base_link, child laser, origin xyz=0 0 0.1 rpy=0 0 0
- joint _right_index_mid: axis 1 0 0 -> -1 0 0
- joint _right_index_tip: axis 1 0 0 -> -1 0 0
- joint _right_middle_mid: axis 1 0 0 -> -1 0 0
- joint _right_middle_tip: axis 1 0 0 -> -1 0 0
- joint _right_pinky_mid: axis 1 0 0 -> -1 0 0
- joint _right_pinky_tip: axis 1 0 0 -> -1 0 0
- joint _right_ring_mid: axis 1 0 0 -> -1 0 0
- joint _right_ring_tip: axis 1 0 0 -> -1 0 0
- joint _right_thumb_mid: axis 1 0 0 -> -1 0 0
- joint _right_thumb_tip: axis 1 0 0 -> -1 0 0
- joint right_index: axis 1 0 0 -> -1 0 0
- joint right_middle: axis 1 0 0 -> -1 0 0
- joint right_pinky: axis 1 0 0 -> -1 0 0
- joint right_ring: axis 1 0 0 -> -1 0 0
- joint right_thumb: axis 1 0 0 -> -1 0 0

Commit message: fix the rotation of lazer

File: urdfs/mc_one.urdf (robot description, URDF)
Before this commit: robot mc_one, 55 links, 57 joints
Joints:
- joint laser_mount: origin xyz=0 0 0.1 rpy=0 0 0 -> xyz=0 0 0.1 rpy=0 0 -1.5707963

Commit message: add imu

File: urdfs/mc_one.urdf (robot description, URDF)
Before this commit: robot mc_one, 55 links, 57 joints
Links:
- added link imu
Joints:
- added joint imu_mount: type fixed, parent base_link, child imu, origin xyz=0 0 0 rpy=0 0 0
