Commit message: isaac full body

File: urdf/mc1.urdf (robot description, URDF)
Before this commit: robot mc1, 19 links, 18 joints
Links:
- added link head, mass 0.6; collision box size=0.195 0.156 0.207; visual mesh filename=package://mc_robot_description/meshes/mc1/head.stl
- added link head_camera_link, mass 0.05; visual box size=0.001 0.001 0.001
- added link head_camera_optical_frame, mass 0.05; visual box size=0.001 0.001 0.001
- added link imu, mass 0.05; visual box size=0.001 0.001 0.001
- added link laser, mass 0.05; visual box size=0.001 0.001 0.001
- added link left_index_base, mass 0.02; visual mesh filename=package://mc_robot_description/meshes/mc1/left_finger_base_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
- added link left_index_mid, mass 0.01; visual mesh filename=package://mc_robot_description/meshes/mc1/left_finger_mid.s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
- added link left_index_tip, mass 0.01; visual mesh filename=package://mc_robot_description/meshes/mc1/left_finger_tip.s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
- added link left_middle_base, mass 0.02; visual mesh filename=package://mc_robot_description/meshes/mc1/left_finger_base_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
- added link left_middle_mid, mass 0.01; visual mesh filename=package://mc_robot_description/meshes/mc1/left_finger_mid.s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
- added link left_middle_tip, mass 0.01; visual mesh filename=package://mc_robot_description/meshes/mc1/left_finger_tip.s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
- added link left_palm, mass 0.2; collision box size=0.101 0.121 0.055; visual mesh filename=package://mc_robot_description/meshes/mc1/left_palm.stl
- added link left_pinky_base, mass 0.02; visual mesh filename=package://mc_robot_description/meshes/mc1/left_finger_base_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
- added link left_pinky_mid, mass 0.01; visual mesh filename=package://mc_robot_description/meshes/mc1/left_finger_mid.s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
- added link left_pinky_tip, mass 0.01; visual mesh filename=package://mc_robot_description/meshes/mc1/left_finger_tip.s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
- added link left_ring_base, mass 0.02; visual mesh filename=package://mc_robot_description/meshes/mc1/left_finger_base_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
- added link left_ring_mid, mass 0.01; visual mesh filename=package://mc_robot_description/meshes/mc1/left_finger_mid.s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
- added link left_ring_tip, mass 0.01; visual mesh filename=package://mc_robot_description/meshes/mc1/left_finger_tip.s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
- added link left_thumb_base, mass 0.02; visual mesh filename=package://mc_robot_description/meshes/mc1/left_thumb_base.s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
- added link left_thumb_mid, mass 0.01; visual mesh filename=package://mc_robot_description/meshes/mc1/left_finger_mid.s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
- added link left_thumb_tip, mass 0.01; visual mesh filename=package://mc_robot_description/meshes/mc1/left_finger_tip.s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
- added link left_wheel, mass 0.5; collision cylinder length=0.05 radius=0.076; visual mesh filename=package://mc_robot_description/meshes/mc1/left_wheel.stl
- added link limit_switch_front, mass 0.05; visual box size=0.001 0.001 0.001
- added link limit_switch_rear, mass 0.05; visual box size=0.001 0.001 0.001
- added link neck, mass 0.2; collision box size=0.1 0.07 0.161; visual mesh filename=package://mc_robot_description/meshes/mc1/neck.stl
- added link pelvis, mass 1.0; collision box size=0.131 0.252 0.149; visual mesh filename=package://mc_robot_description/meshes/mc1/pelvis.stl
- added link right_index_base, mass 0.02; visual mesh filename=package://mc_robot_description/meshes/mc1/right_finger_base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
- added link right_index_mid, mass 0.01; visual mesh filename=package://mc_robot_description/meshes/mc1/right_finger_mid.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
- added link right_index_tip, mass 0.01; visual mesh filename=package://mc_robot_description/meshes/mc1/right_finger_tip.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
- added link right_middle_base, mass 0.02; visual mesh filename=package://mc_robot_description/meshes/mc1/right_finger_base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
- added link right_middle_mid, mass 0.01; visual mesh filename=package://mc_robot_description/meshes/mc1/right_finger_mid.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
- added link right_middle_tip, mass 0.01; visual mesh filename=package://mc_robot_description/meshes/mc1/right_finger_tip.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
- added link right_palm, mass 0.2; collision box size=0.101 0.121 0.055; visual mesh filename=package://mc_robot_description/meshes/mc1/right_palm.stl
- added link right_pinky_base, mass 0.02; visual mesh filename=package://mc_robot_description/meshes/mc1/right_finger_base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
- added link right_pinky_mid, mass 0.01; visual mesh filename=package://mc_robot_description/meshes/mc1/right_finger_mid.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
- added link right_pinky_tip, mass 0.01; visual mesh filename=package://mc_robot_description/meshes/mc1/right_finger_tip.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
- added link right_ring_base, mass 0.02; visual mesh filename=package://mc_robot_description/meshes/mc1/right_finger_base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
- added link right_ring_mid, mass 0.01; visual mesh filename=package://mc_robot_description/meshes/mc1/right_finger_mid.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
- added link right_ring_tip, mass 0.01; visual mesh filename=package://mc_robot_description/meshes/mc1/right_finger_tip.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
- added link right_thumb_base, mass 0.02; visual mesh filename=package://mc_robot_description/meshes/mc1/right_thumb_base.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
- added link right_thumb_mid, mass 0.01; visual mesh filename=package://mc_robot_description/meshes/mc1/right_finger_mid.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
- added link right_thumb_tip, mass 0.01; visual mesh filename=package://mc_robot_description/meshes/mc1/right_finger_tip.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
- added link right_wheel, mass 0.5; collision cylinder length=0.05 radius=0.076; visual mesh filename=package://mc_robot_description/meshes/mc1/right_wheel.stl
- added link tof_front_left, mass 0.05; visual box size=0.001 0.001 0.001
- added link tof_front_right, mass 0.05; visual box size=0.001 0.001 0.001
- added link tof_rear_left, mass 0.05; visual box size=0.001 0.001 0.001
- added link tof_rear_right, mass 0.05; visual box size=0.001 0.001 0.001
- added link torso, mass 2.0; collision box size=0.154 0.22 0.347; visual mesh filename=package://mc_robot_description/meshes/mc1/torso.stl
- added link upper_legs, mass 1.5; collision box size=0.181 0.268 0.294; visual mesh filename=package://mc_robot_description/meshes/mc1/upper_legs.stl
- added link waist_base_link, mass 0.670115; collision mesh filename=package://mc_robot_description/meshes/mc1/base_link.stl; visual mesh filename=package://mc_robot_description/meshes/mc1/base_link.stl
- link base_link: mass 0.670115 -> 5.0; geometry collision box size=0.411 0.45 0.321; visual mesh filename=package://mc_robot_description/meshes/mc1/base.stl
Joints:
- added joint _left_index_mid: type revolute, parent left_index_base, child left_index_mid, origin xyz=0 0.0198 -0.0028 rpy=0 0 0, axis 1 0 0, limit lower=-1.1 upper=0.0 effort=2 velocity=5, mimic joint=left_index multiplier=1 offset=0
- added joint _left_index_tip: type revolute, parent left_index_mid, child left_index_tip, origin xyz=-0.004 0.02 0 rpy=0 0 0, axis 1 0 0, limit lower=-1.1 upper=0.0 effort=2 velocity=5, mimic joint=left_index multiplier=1 offset=0
- added joint _left_middle_mid: type revolute, parent left_middle_base, child left_middle_mid, origin xyz=0 0.0198 -0.0028 rpy=0 0 0, axis 1 0 0, limit lower=-1.1 upper=0.0 effort=2 velocity=5, mimic joint=left_middle multiplier=1 offset=0
- added joint _left_middle_tip: type revolute, parent left_middle_mid, child left_middle_tip, origin xyz=0.004 0.02 0 rpy=0 0 0, axis 1 0 0, limit lower=-1.1 upper=0.0 effort=2 velocity=5, mimic joint=left_middle multiplier=1 offset=0
- added joint _left_pinky_mid: type revolute, parent left_pinky_base, child left_pinky_mid, origin xyz=0 0.0198 -0.0028 rpy=0 0 0, axis 1 0 0, limit lower=-1.1 upper=0.0 effort=2 velocity=5, mimic joint=left_pinky multiplier=1 offset=0
- added joint _left_pinky_tip: type revolute, parent left_pinky_mid, child left_pinky_tip, origin xyz=0.004 0.02 0 rpy=0 0 0, axis 1 0 0, limit lower=-1.1 upper=0.0 effort=2 velocity=5, mimic joint=left_pinky multiplier=1 offset=0
- added joint _left_ring_mid: type revolute, parent left_ring_base, child left_ring_mid, origin xyz=0 0.0199 -0.0028 rpy=0 0 0, axis 1 0 0, limit lower=-1.1 upper=0.0 effort=2 velocity=5, mimic joint=left_ring multiplier=1 offset=0
- added joint _left_ring_tip: type revolute, parent left_ring_mid, child left_ring_tip, origin xyz=-0.004 0.02 0 rpy=0 0 0, axis 1 0 0, limit lower=-1.1 upper=0.0 effort=2 velocity=5, mimic joint=left_ring multiplier=1 offset=0
- added joint _left_thumb_mid: type revolute, parent left_thumb_base, child left_thumb_mid, origin xyz=0 0.0185 -0.007 rpy=0 0 0, axis 1 0 0, limit lower=-1.1 upper=0.0 effort=2 velocity=5, mimic joint=left_thumb multiplier=1 offset=0
- added joint _left_thumb_tip: type revolute, parent left_thumb_mid, child left_thumb_tip, origin xyz=-0.004 0.0201 0 rpy=0 0 0, axis 1 0 0, limit lower=-1.1 upper=0.0 effort=2 velocity=5, mimic joint=left_thumb multiplier=1 offset=0
- added joint _right_index_mid: type revolute, parent right_index_base, child right_index_mid, origin xyz=0 -0.0198 -0.0028 rpy=0 0 0, axis -1 0 0, limit lower=0.0 upper=1.1 effort=2 velocity=5, mimic joint=right_index multiplier=1 offset=0
- added joint _right_index_tip: type revolute, parent right_index_mid, child right_index_tip, origin xyz=-0.004 -0.02 0 rpy=0 0 0, axis -1 0 0, limit lower=0.0 upper=1.1 effort=2 velocity=5, mimic joint=right_index multiplier=1 offset=0
- added joint _right_middle_mid: type revolute, parent right_middle_base, child right_middle_mid, origin xyz=0 -0.0198 -0.0028 rpy=0 0 0, axis -1 0 0, limit lower=0.0 upper=1.1 effort=2 velocity=5, mimic joint=right_middle multiplier=1 offset=0
- added joint _right_middle_tip: type revolute, parent right_middle_mid, child right_middle_tip, origin xyz=0.004 -0.02 0 rpy=0 0 0, axis -1 0 0, limit lower=0.0 upper=1.1 effort=2 velocity=5, mimic joint=right_middle multiplier=1 offset=0
- added joint _right_pinky_mid: type revolute, parent right_pinky_base, child right_pinky_mid, origin xyz=0 -0.0198 -0.0028 rpy=0 0 0, axis -1 0 0, limit lower=0.0 upper=1.1 effort=2 velocity=5, mimic joint=right_pinky multiplier=1 offset=0
- added joint _right_pinky_tip: type revolute, parent right_pinky_mid, child right_pinky_tip, origin xyz=0.004 -0.02 0 rpy=0 0 0, axis -1 0 0, limit lower=0.0 upper=1.1 effort=2 velocity=5, mimic joint=right_pinky multiplier=1 offset=0
- added joint _right_ring_mid: type revolute, parent right_ring_base, child right_ring_mid, origin xyz=0 -0.0199 -0.0028 rpy=0 0 0, axis -1 0 0, limit lower=0.0 upper=1.1 effort=2 velocity=5, mimic joint=right_ring multiplier=1 offset=0
- added joint _right_ring_tip: type revolute, parent right_ring_mid, child right_ring_tip, origin xyz=-0.004 -0.02 0 rpy=0 0 0, axis -1 0 0, limit lower=0.0 upper=1.1 effort=2 velocity=5, mimic joint=right_ring multiplier=1 offset=0
- added joint _right_thumb_mid: type revolute, parent right_thumb_base, child right_thumb_mid, origin xyz=0 -0.0185 -0.0075 rpy=0 0 0, axis -1 0 0, limit lower=0.0 upper=1.1 effort=2 velocity=5, mimic joint=right_thumb multiplier=1 offset=0
- added joint _right_thumb_tip: type revolute, parent right_thumb_mid, child right_thumb_tip, origin xyz=-0.004 -0.02 0.0 rpy=0 0 0, axis -1 0 0, limit lower=0.0 upper=1.1 effort=2 velocity=5, mimic joint=right_thumb multiplier=1 offset=0
- added joint head_camera_joint: type fixed, parent head, child head_camera_link, origin xyz=0.09 0 0.03 rpy=0 0 0
- added joint head_camera_optical_joint: type fixed, parent head_camera_link, child head_camera_optical_frame, origin xyz=0 0 0 rpy=-1.5707963267949 0 -1.5707963267949
- added joint head_nod: type revolute, parent neck, child head, origin xyz=0.00698 0 0.1 rpy=0 0 0, axis 0 1 0, limit lower=-0.6981317 upper=0.4363323 effort=10 velocity=2
- added joint hips: type revolute, parent upper_legs, child pelvis, origin xyz=-0.10564 0 0.21708 rpy=0 0 0, axis 0 1 0, limit lower=-0.366519142918809 upper=1.5707963267949 effort=50 velocity=2, mimic joint=knees multiplier=-1 offset=0
- added joint imu_mount: type fixed, parent base_link, child imu, origin xyz=0 0 0 rpy=0 0 0
- added joint knees: type revolute, parent base_link, child upper_legs, origin xyz=-0.0275 0 0.226 rpy=0 0 0, axis 0 1 0, limit lower=-1.5707963267949 upper=0.366519142918809 effort=50 velocity=2
- added joint laser_mount: type fixed, parent base_link, child laser, origin xyz=0 0 0.1 rpy=0 0 -1.5707963267949
- added joint left_index: type revolute, parent left_palm, child left_index_base, origin xyz=0.0277 0.1061 -0.004 rpy=0 0 -0.1047198, axis 1 0 0, limit lower=-1.1 upper=0.0 effort=2 velocity=5
- added joint left_middle: type revolute, parent left_palm, child left_middle_base, origin xyz=0.002 0.111 -0.004 rpy=0 0 -0.0349066, axis 1 0 0, limit lower=-1.1 upper=0.0 effort=2 velocity=5
- added joint left_palm_joint: type fixed, parent left_arm_tcp, child left_palm, origin xyz=0 0 0 rpy=1.5707963267949 0 0
- added joint left_pinky: type revolute, parent left_palm, child left_pinky_base, origin xyz=-0.0406 0.1061 -0.004 rpy=0 0 0.1047198, axis 1 0 0, limit lower=-1.1 upper=0.0 effort=2 velocity=5
- added joint left_ring: type revolute, parent left_palm, child left_ring_base, origin xyz=-0.0109 0.111 -0.004 rpy=0 0 0.0349066, axis 1 0 0, limit lower=-1.1 upper=0.0 effort=2 velocity=5
- added joint left_thumb: type revolute, parent left_palm, child left_thumb_base, origin xyz=0.0446 0.0484 -0.019 rpy=0 0 -2.268928, axis 1 0 0, limit lower=-1.1 upper=0.0 effort=2 velocity=5
- added joint left_wheel: type continuous, parent base_link, child left_wheel, origin xyz=0 0.182 0 rpy=0 0 0, axis 0 1 0, limit effort=10 velocity=34.5
- added joint limit_switch_front_mount: type fixed, parent base_link, child limit_switch_front, origin xyz=0.07 0 0 rpy=0 0 0
- added joint limit_switch_rear_mount: type fixed, parent base_link, child limit_switch_rear, origin xyz=-0.335 0 0 rpy=0 0 3.14159265358979
- added joint neck_turn: type revolute, parent torso, child neck, origin xyz=0.00096 0 0.38092 rpy=0 0 0, axis 0 0 1, limit lower=-1.3962634 upper=1.3962634 effort=10 velocity=2
- added joint right_index: type revolute, parent right_palm, child right_index_base, origin xyz=0.0277 -0.1101 -0.004 rpy=0 0 0.1047198, axis -1 0 0, limit lower=0.0 upper=1.1 effort=2 velocity=5
- added joint right_middle: type revolute, parent right_palm, child right_middle_base, origin xyz=0.002 -0.115 -0.004 rpy=0 0 0.0349066, axis -1 0 0, limit lower=0.0 upper=1.1 effort=2 velocity=5
- added joint right_palm_joint: type fixed, parent right_arm_tcp, child right_palm, origin xyz=0 0 0 rpy=-1.5707963267949 0 0
- added joint right_pinky: type revolute, parent right_palm, child right_pinky_base, origin xyz=-0.0406 -0.1101 -0.004 rpy=0 0 -0.1047198, axis -1 0 0, limit lower=0.0 upper=1.1 effort=2 velocity=5
- added joint right_ring: type revolute, parent right_palm, child right_ring_base, origin xyz=-0.0109 -0.115 -0.004 rpy=0 0 -0.0349066, axis -1 0 0, limit lower=0.0 upper=1.1 effort=2 velocity=5
- added joint right_thumb: type revolute, parent right_palm, child right_thumb_base, origin xyz=0.0446 -0.0525 -0.019 rpy=0 0 2.268928, axis -1 0 0, limit lower=0.0 upper=1.1 effort=2 velocity=5
- added joint right_wheel: type continuous, parent base_link, child right_wheel, origin xyz=0 -0.182 0 rpy=0 0 0, axis 0 1 0, limit effort=10 velocity=34.5
- added joint tof_front_left_mount: type fixed, parent base_link, child tof_front_left, origin xyz=0.06 0.20 -0.05 rpy=0 1.5707963267949 0
- added joint tof_front_right_mount: type fixed, parent base_link, child tof_front_right, origin xyz=0.06 -0.20 -0.05 rpy=0 1.5707963267949 0
- added joint tof_rear_left_mount: type fixed, parent base_link, child tof_rear_left, origin xyz=-0.32 0.20 -0.05 rpy=0 1.5707963267949 0
- added joint tof_rear_right_mount: type fixed, parent base_link, child tof_rear_right, origin xyz=-0.32 -0.20 -0.05 rpy=0 1.5707963267949 0
- added joint torso_shell_joint: type fixed, parent waist_link, child torso, origin xyz=0 0 0.28 rpy=0 0 0
- added joint waist_base_joint: type fixed, parent pelvis, child waist_base_link, origin xyz=0 0 0.10 rpy=0 0 0
- joint left_arm_joint_1: origin xyz=0 0.0443862 0.282191 rpy=0 -1.309 -1.5707963267949 -> xyz=0.00084 0.09165 0.33902 rpy=0 -1.309 -1.5707963267949; parent waist_link -> torso
- joint right_arm_joint_1: origin xyz=0 -0.0443877 0.282191 rpy=0 -1.309 1.5707963267949 -> xyz=0.00084 -0.09165 0.33902 rpy=0 -1.309 1.5707963267949; parent waist_link -> torso
- joint waist_joint: parent base_link -> waist_base_link

Commit message: update urdf now everything is right

File: urdf/mc1.urdf (robot description, URDF)
Before this commit: robot mc1, 69 links, 68 joints
Links:
- removed link head_camera_optical_frame
- removed link realsense_link
- removed link realsense_mount_link
- removed link realsense_optical_frame
- removed link waist_base_link
- removed link waist_link
- added link chest_camera_link, mass 0.08; collision box size=0.05 0.09 0.03; visual mesh filename=package://mc_robot_description/meshes/mc1/camera.stl
- added link chest_camera_sensor, mass 0.05; visual box size=0.001 0.001 0.001
Joints:
- removed joint head_camera_optical_joint
- removed joint realsense_mount_joint
- removed joint realsense_optical_joint
- removed joint realsense_pitch_joint
- removed joint torso_shell_joint
- removed joint waist_base_joint
- removed joint waist_joint
- added joint camera_sensor_joint: type fixed, parent chest_camera_link, child chest_camera_sensor, origin xyz=0.03 0 0 rpy=0 0 0
- added joint chest_camera: type revolute, parent torso, child chest_camera_link, origin xyz=0.048749 0 0.336 rpy=0 0 0, axis 0 1 0, limit lower=-0.4 upper=0.4 effort=2 velocity=1
- added joint torso_rotate: type revolute, parent pelvis, child torso, origin xyz=0 0 0 rpy=0 0 0, axis 0 0 1, limit lower=-1.3963 upper=1.3963 effort=50 velocity=2
- joint _right_index_mid: axis -1 0 0 -> 1 0 0
- joint _right_index_tip: axis -1 0 0 -> 1 0 0
- joint _right_middle_mid: axis -1 0 0 -> 1 0 0
- joint _right_middle_tip: axis -1 0 0 -> 1 0 0
- joint _right_pinky_mid: axis -1 0 0 -> 1 0 0
- joint _right_pinky_tip: axis -1 0 0 -> 1 0 0
- joint _right_ring_mid: axis -1 0 0 -> 1 0 0
- joint _right_ring_tip: axis -1 0 0 -> 1 0 0
- joint _right_thumb_mid: axis -1 0 0 -> 1 0 0
- joint _right_thumb_tip: axis -1 0 0 -> 1 0 0
- joint head_camera_joint: origin xyz=0.09 0 0.03 rpy=0 0 0 -> xyz=0.09 0 0.06 rpy=0 0 0
- joint left_arm_tcp_joint: origin xyz=0 0.1 0 rpy=-1.5707963267949 0 0 -> xyz=0 0.075 0 rpy=-1.5707963267949 0 0
- joint left_palm_joint: origin xyz=0 0 0 rpy=1.5707963267949 0 0 -> xyz=0 0 0 rpy=1.570796327 0 -1.570796327
- joint limit_switch_front_mount: origin xyz=0.07 0 0 rpy=0 0 0 -> xyz=0.12 0 0 rpy=0 0 0
- joint right_arm_tcp_joint: origin xyz=0 0.1 0 rpy=-1.5707963267949 0 0 -> xyz=0 0.075 0 rpy=-1.5707963267949 0 0
- joint right_index: axis -1 0 0 -> 1 0 0
- joint right_middle: axis -1 0 0 -> 1 0 0
- joint right_palm_joint: origin xyz=0 0 0 rpy=-1.5707963267949 0 0 -> xyz=0 0 0 rpy=-1.570796327 0 1.570796327
- joint right_pinky: axis -1 0 0 -> 1 0 0
- joint right_ring: axis -1 0 0 -> 1 0 0
- joint right_thumb: axis -1 0 0 -> 1 0 0
- joint tof_front_left_mount: origin xyz=0.06 0.20 -0.05 rpy=0 1.5707963267949 0 -> xyz=0.11 0.20 -0.031 rpy=0 1.5707963267949 0
- joint tof_front_right_mount: origin xyz=0.06 -0.20 -0.05 rpy=0 1.5707963267949 0 -> xyz=0.11 -0.20 -0.031 rpy=0 1.5707963267949 0
- joint tof_rear_left_mount: origin xyz=-0.32 0.20 -0.05 rpy=0 1.5707963267949 0 -> xyz=-0.32 0.13 -0.031 rpy=0 1.5707963267949 0
- joint tof_rear_right_mount: origin xyz=-0.32 -0.20 -0.05 rpy=0 1.5707963267949 0 -> xyz=-0.32 -0.13 -0.031 rpy=0 1.5707963267949 0

Commit message: add universal wheel

File: urdf/mc1.urdf (robot description, URDF)
Before this commit: robot mc1, 65 links, 64 joints
Links:
- link base_link: geometry collision box size=0.411 0.45 0.321; collision sphere radius=0.0155

Commit message: update

File: urdf/mc1.urdf (robot description, URDF)
Before this commit: robot mc1, 65 links, 64 joints
Links:
- link left_wheel: geometry collision cylinder length=0.05 radius=0.05; visual mesh filename=package://mc_robot_description/meshes/mc1/left_wheel.stl scale=0.656168 1 0.656168
- link right_wheel: geometry collision cylinder length=0.05 radius=0.05; visual mesh filename=package://mc_robot_description/meshes/mc1/right_wheel.stl scale=0.656168 1 0.656168
Joints:
- joint imu_mount: origin xyz=0 0 0 rpy=0 0 0 -> xyz=0 0 0.026 rpy=0 0 0
- joint knees: origin xyz=-0.0275 0 0.226 rpy=0 0 0 -> xyz=-0.0275 0 0.252 rpy=0 0 0
- joint laser_mount: origin xyz=0 0 0.1 rpy=0 0 -1.5707963267949 -> xyz=0 0 0.126 rpy=0 0 -1.5707963267949
- joint left_wheel: origin xyz=0 0.182 0 rpy=0 0 0 -> xyz=0 0.165 0 rpy=0 0 0
- joint limit_switch_front_mount: origin xyz=0.12 0 0 rpy=0 0 0 -> xyz=0.12 0 0.026 rpy=0 0 0
- joint limit_switch_rear_mount: origin xyz=-0.335 0 0 rpy=0 0 3.14159265358979 -> xyz=-0.335 0 0.026 rpy=0 0 3.14159265358979
- joint right_wheel: origin xyz=0 -0.182 0 rpy=0 0 0 -> xyz=0 -0.165 0 rpy=0 0 0
- joint tof_front_left_mount: origin xyz=0.11 0.20 -0.031 rpy=0 1.5707963267949 0 -> xyz=0.11 0.20 -0.005 rpy=0 1.5707963267949 0
- joint tof_front_right_mount: origin xyz=0.11 -0.20 -0.031 rpy=0 1.5707963267949 0 -> xyz=0.11 -0.20 -0.005 rpy=0 1.5707963267949 0
- joint tof_rear_left_mount: origin xyz=-0.32 0.13 -0.031 rpy=0 1.5707963267949 0 -> xyz=-0.32 0.13 -0.005 rpy=0 1.5707963267949 0
- joint tof_rear_right_mount: origin xyz=-0.32 -0.13 -0.031 rpy=0 1.5707963267949 0 -> xyz=-0.32 -0.13 -0.005 rpy=0 1.5707963267949 0

Commit message: update

File: urdf/mc1.urdf (robot description, URDF)
Before this commit: robot mc1, 65 links, 64 joints
Links:
- link base_link: geometry collision box size=0.411 0.45 0.321; collision sphere radius=0.006

Commit message: update

File: urdf/mc1.urdf (robot description, URDF)
Before this commit: robot mc1, 65 links, 64 joints
Links:
- link base_link: geometry collision box size=0.411 0.45 0.321; collision sphere radius=0.01
Joints:
- joint left_arm_joint_1: origin xyz=0.00084 0.09165 0.33902 rpy=0 -1.309 -1.5707963267949 -> xyz=0.00084 0.03165 0.33902 rpy=0 -1.309 -1.5707963267949
- joint left_palm_joint: origin xyz=0 0 0 rpy=1.570796327 0 -1.570796327 -> xyz=0 0 -0.03 rpy=1.570796327 0 -1.570796327
- joint right_arm_joint_1: origin xyz=0.00084 -0.09165 0.33902 rpy=0 -1.309 1.5707963267949 -> xyz=0.00084 -0.03165 0.33902 rpy=0 -1.309 1.5707963267949
- joint right_palm_joint: origin xyz=0 0 0 rpy=-1.570796327 0 1.570796327 -> xyz=0 0 -0.03 rpy=-1.570796327 0 1.570796327

Commit message: update

File: urdf/mc1.urdf (robot description, URDF)
Before this commit: robot mc1, 65 links, 64 joints
Joints:
- joint _left_thumb_mid: origin xyz=0 0.0185 -0.007 rpy=0 0 0 -> xyz=0 0.0185 -0.0075 rpy=0 0 0
- joint _left_thumb_tip: origin xyz=-0.004 0.0201 0 rpy=0 0 0 -> xyz=-0.004 0.02 0 rpy=0 0 0
- joint left_index: origin xyz=0.0277 0.1061 -0.004 rpy=0 0 -0.1047198 -> xyz=0.0277 0.1101 -0.004 rpy=0 0 -0.1047198
- joint left_middle: origin xyz=0.002 0.111 -0.004 rpy=0 0 -0.0349066 -> xyz=0.002 0.115 -0.004 rpy=0 0 -0.0349066
- joint left_pinky: origin xyz=-0.0406 0.1061 -0.004 rpy=0 0 0.1047198 -> xyz=-0.0406 0.1101 -0.004 rpy=0 0 0.1047198
- joint left_ring: origin xyz=-0.0109 0.111 -0.004 rpy=0 0 0.0349066 -> xyz=-0.0109 0.115 -0.004 rpy=0 0 0.0349066
- joint left_thumb: origin xyz=0.0446 0.0484 -0.019 rpy=0 0 -2.268928 -> xyz=0.0446 0.0525 -0.019 rpy=0 0 -2.268928
